Commit message: change leo_simulation -> simulation_package, slam capability semi-complete

File: src/hardware_package/urdf/robot.urdf (robot description, URDF)
Before this commit: robot leo, 15 links, 14 joints
Links:
- removed link antenna_link
- removed link camera_frame
- removed link camera_optical_frame
- removed link imu_frame
- removed link rocker_L_link
- removed link rocker_R_link
- link base_link: geometry collision mesh filename=package://hardware_package/meshes/Chass_outline.stl; visual mesh filename=package://hardware_package/meshes/Chassis.dae scale=1 1 1
- link lidar_link: geometry visual mesh filename=package://hardware_package/meshes/Generic_100mm_lidar.stl scale=1 1 1
- link sled_link: geometry visual mesh filename=package://hardware_package/meshes/Rover_mounts_v1.stl scale=0.001 0.001 0.001
- link wheel_FL_link: mass 0.283642 -> None; geometry collision cylinder length=0.066 radius=0.065; visual mesh filename=package://hardware_package/meshes/WheelA.dae
- link wheel_FR_link: mass 0.283642 -> None; geometry collision cylinder length=0.066 radius=0.065; visual mesh filename=package://hardware_package/meshes/WheelA.dae
- link wheel_RL_link: mass 0.283642 -> None; geometry collision cylinder length=0.066 radius=0.065; visual mesh filename=package://hardware_package/meshes/WheelA.dae
- link wheel_RR_link: mass 0.283642 -> None; geometry collision cylinder length=0.066 radius=0.065; visual mesh filename=package://hardware_package/meshes/WheelA.dae
Joints:
- removed joint antenna_joint
- removed joint base_joint
- removed joint camera_joint
- removed joint camera_optical_joint
- removed joint imu_joint
- removed joint rocker_L_joint
- removed joint rocker_R_joint
- removed joint wheel_FL_joint
- removed joint wheel_FR_joint
- removed joint wheel_RL_joint
- removed joint wheel_RR_joint
- added joint base_FL_joint: type continuous, parent base_link, child wheel_FL_link, origin xyz=0.148 -0.1795 0 rpy=0 0 0
- added joint base_FR_joint: type continuous, parent base_link, child wheel_FR_link, origin xyz=0.148 0.1795 0 rpy=0 0 0
- added joint base_RL_joint: type continuous, parent base_link, child wheel_RL_link, origin xyz=-0.148 -0.1795 0 rpy=0 0 0
- added joint base_RR_joint: type continuous, parent base_link, child wheel_RR_link, origin xyz=-0.148 0.1795 0 rpy=0 0 0
- added joint base_footprint_joint: type fixed, parent base_footprint, child base_link, origin xyz=0 0 0 rpy=0 0 0
