Commit message: fixes and rqt graphs

File: src/hardware_package/urdf/leo.urdf.xacro (robot description, xacro)
@@ -3,10 +3,10 @@
        name="leo">
   <xacro:arg name="mecanum_wheels" default="false"/>
-  <xacro:include filename="$(find leo_description)/urdf/macros.xacro"/>
+  <xacro:include filename="./macros.xacro"/>
   <xacro:leo mecanum_wheels="$(arg mecanum_wheels)"/>
   <link name="lidar_link">
      <visual>
           <geometry>
-             <mesh filename="package://leo_simulation/meshes/Generic_100mm_lidar.stl" scale="1 1 1"/>
+             <mesh filename="../meshes/Generic_100mm_lidar.stl" scale="1 1 1"/>
           </geometry>
           <material name="red">
@@ -20,5 +20,5 @@
       <origin xyz="0.0 0.0 0.0" rpy="0.0 0.0 0.0"/>
       <geometry>
-         <mesh filename="package://leo_simulation/meshes/Rover_mounts_v1.stl" scale="0.001 0.001 0.001" />
+         <mesh filename="../meshes/Rover_mounts_v1.stl" scale="0.001 0.001 0.001" />
       </geometry>
       <material name="blue">

Commit message: navigation nearly working

File: src/hardware_package/urdf/leo.urdf.xacro (robot description, xacro)
@@ -41,5 +41,5 @@
      <parent link="base_link"/>
      <child link="lidar_link"/>
-     <origin xyz="0.02 0 0.05" rpy="0 0 0" />
+     <origin xyz="0.02 0 0.05" rpy="0 0 3.14" />
   </joint>
   <joint name="sled_base_joint" type="fixed">

Commit message: merge problems have caused this

File: src/hardware_package/urdf/leo.urdf.xacro (robot description, xacro)
@@ -41,5 +41,5 @@
      <parent link="base_link"/>
      <child link="lidar_link"/>
-     <origin xyz="0.02 0 0.05" rpy="0 0 3.14" />
+     <origin xyz="0.02 0 0.05" rpy="0 0 -3.14" />
   </joint>
   <joint name="sled_base_joint" type="fixed">

File: src/hardware_package/urdf/leo_rover.urdf.xacro (robot description, xacro)
@@ -189,5 +189,5 @@
         <parent link="base_link"/>
         <child link="lidar_link"/>
-        <origin xyz="0.02 0.001 0.05" rpy="0 0 -1.57" />
+        <origin xyz="0.02 0.001 0.05" rpy="0 0 -3.14" />
     </joint>
     <joint name="sled_base_joint" type="fixed">

Commit message: update

File: src/hardware_package/urdf/leo.urdf.xacro (robot description, xacro)
@@ -2,11 +2,15 @@
 <robot xmlns:xacro="http://www.ros.org/wiki/xacro"
        name="leo">
-  <xacro:arg name="mecanum_wheels" default="false"/>
-  <xacro:include filename="./macros.xacro"/>
-  <xacro:leo mecanum_wheels="$(arg mecanum_wheels)"/>
+   <xacro:arg name="mecanum_wheels" default="false"/>
+   <xacro:include filename="./macros.xacro"/>
+   <xacro:include filename="$(find realsense2_description)/urdf/_d435i.urdf.xacro"/>
+   <xacro:leo mecanum_wheels="$(arg mecanum_wheels)"/>
+   <xacro:sensor_d435i parent="base_link" name="_camera">
+      <origin xyz="0.155 0 0.2" rpy="0 0 0"/>
+   </xacro:sensor_d435i>
   <link name="lidar_link">
      <visual>
           <geometry>
-             <mesh filename="../meshes/Generic_100mm_lidar.stl" scale="1 1 1"/>
+             <mesh filename="package://leo_description/models/Generic_100mm_lidar.stl" scale="1 1 1"/>
           </geometry>
           <material name="red">
@@ -20,5 +24,5 @@
       <origin xyz="0.0 0.0 0.0" rpy="0.0 0.0 0.0"/>
       <geometry>
-         <mesh filename="../meshes/Rover_mounts_v1.stl" scale="0.001 0.001 0.001" />
+         <mesh filename="package://leo_description/models/Rover_mounts_v1.stl" scale="0.001 0.001 0.001" />
       </geometry>
       <material name="blue">
@@ -27,9 +31,9 @@
    </visual>
   </link>
-  <link name="depth_camera_link">
+  <!-- <link name="depth_camera_link">
    <visual name="">
       <origin xyz="0 0 0" rpy="0.0 0.0 0.0"/>
       <geometry>
-         <box size="0.090 0.025 0.025"/>
+         <box size="0.025 0.090 0.025"/>
       </geometry>
       <material name="cyan">
@@ -37,5 +41,5 @@
       </material>
    </visual>
-  </link>
+  </link> -->
   <joint name="lidar_base_joint" type="fixed">
      <parent link="base_link"/>
@@ -48,8 +52,8 @@
       <origin xyz="0 0 -0.02" rpy="0 0 1.57" />
   </joint>
-  <joint name="depth_camera_base_joint" type="fixed">
+  <!-- <joint name="depth_camera_base_joint" type="fixed">
       <parent link="base_link"/>
       <child link="depth_camera_link"/>
-      <origin xyz="0.155 0 0" rpy="-1.57 0 -1.57" />
-  </joint>
+      <origin xyz="0.155 0 0.2" rpy="-3.14 0 -3.14" />
+  </joint> -->
 </robot>

File: src/hardware_package/urdf/leo_rover.urdf.xacro (robot description, xacro)
@@ -199,5 +199,5 @@
         <parent link="base_link"/>
         <child link="depth_camera_link"/>
-        <origin xyz="0.155 0 0" rpy="-1.57 0 -1.57" />
+        <origin xyz="0.155 0 0.2" rpy="0 0 0" />
     </joint>
 </robot>
