Commit message: fixed inverted odom -> base_link tf in simulation

File: src/simulation_package/urdf/leo_sim.urdf.xacro (robot description, xacro)
@@ -169,5 +169,5 @@
         <parent link="base_link"/>
         <child link="wheel_FR_link"/>
-        <origin xyz="${wheelbase/2} -${wheel_separation/2} -0.1" rpy="-1.5707 0 0" />
+        <origin xyz="${wheelbase/2} -${wheel_separation/2} -0.1" rpy="1.5707 0 0" />
         <axis xyz="0 0 1" />
     </joint>
@@ -175,5 +175,5 @@
         <parent link="base_link"/>
         <child link="wheel_FL_link"/>
-        <origin xyz="${wheelbase/2} ${wheel_separation/2} -0.1" rpy="-1.5707 0 0" />
+        <origin xyz="${wheelbase/2} ${wheel_separation/2} -0.1" rpy="1.5707 0 0" />
         <axis xyz="0 0 1" />
     </joint>
@@ -181,5 +181,5 @@
         <parent link="base_link"/>
         <child link="wheel_RR_link"/>
-        <origin xyz="-${wheelbase/2} -${wheel_separation/2} -0.1" rpy="-1.5707 0 0" />
+        <origin xyz="-${wheelbase/2} -${wheel_separation/2} -0.1" rpy="1.5707 0 0" />
         <axis xyz="0 0 1" />
     </joint>
@@ -187,5 +187,5 @@
         <parent link="base_link"/>
         <child link="wheel_RL_link"/>
-        <origin xyz="-${wheelbase/2} ${wheel_separation/2} -0.1" rpy="-1.5707 0 0" />
+        <origin xyz="-${wheelbase/2} ${wheel_separation/2} -0.1" rpy="1.5707 0 0" />
         <axis xyz="0 0 1" />
     </joint>
@@ -223,6 +223,6 @@
       <!-- Wheel Joints -->
       <left_joint>base_FL_joint</left_joint>
+      <left_joint>base_RL_joint</left_joint>
       <right_joint>base_FR_joint</right_joint>
-      <left_joint>base_RL_joint</left_joint>
       <right_joint>base_RR_joint</right_joint>
       <!-- Kinematics -->

Commit message: started work on nav to object

File: src/simulation_package/urdf/leo_sim.urdf.xacro (robot description, xacro)
@@ -169,5 +169,5 @@
         <parent link="base_link"/>
         <child link="wheel_FR_link"/>
-        <origin xyz="${wheelbase/2} -${wheel_separation/2} -0.1" rpy="1.5707 0 0" />
+        <origin xyz="${wheelbase/2} -${wheel_separation/2} -0.1" rpy="-1.5707 0 0" />
         <axis xyz="0 0 1" />
     </joint>
@@ -175,5 +175,5 @@
         <parent link="base_link"/>
         <child link="wheel_FL_link"/>
-        <origin xyz="${wheelbase/2} ${wheel_separation/2} -0.1" rpy="1.5707 0 0" />
+        <origin xyz="${wheelbase/2} ${wheel_separation/2} -0.1" rpy="-1.5707 0 0" />
         <axis xyz="0 0 1" />
     </joint>
@@ -181,5 +181,5 @@
         <parent link="base_link"/>
         <child link="wheel_RR_link"/>
-        <origin xyz="-${wheelbase/2} -${wheel_separation/2} -0.1" rpy="1.5707 0 0" />
+        <origin xyz="-${wheelbase/2} -${wheel_separation/2} -0.1" rpy="-1.5707 0 0" />
         <axis xyz="0 0 1" />
     </joint>
@@ -187,5 +187,5 @@
         <parent link="base_link"/>
         <child link="wheel_RL_link"/>
-        <origin xyz="-${wheelbase/2} ${wheel_separation/2} -0.1" rpy="1.5707 0 0" />
+        <origin xyz="-${wheelbase/2} ${wheel_separation/2} -0.1" rpy="-1.5707 0 0" />
         <axis xyz="0 0 1" />
     </joint>

Commit message: work on simulation

File: src/simulation_package/urdf/leo_sim.urdf.xacro (robot description, xacro)
@@ -6,4 +6,8 @@
     <xacro:property name="wheel_thickness" value="0.066" />
     <xacro:property name="pi" value="3.14159" />
+    <xacro:include filename="$(find realsense2_description)/urdf/_d435i.urdf.xacro"/>
+    <!-- <xacro:sensor_d435i parent="base_link" name="camera_camera">
+      <origin xyz="0 0 0" rpy="0 0 0"/>
+    </xacro:sensor_d435i> -->
     <!-- Materials -->
     <material name="black">
@@ -151,9 +155,9 @@
         </visual>
     </link>
-    <link name="depth_camera_link">
+    <link name="camera_camera_link">
         <visual>
             <origin xyz="0 0 0" rpy="0.0 0.0 0.0"/>
             <geometry>
-                <box size="0.090 0.025 0.025"/>
+                <box size="0.025 0.090 0.025"/>
             </geometry>
             <material name="cyan" />
@@ -200,8 +204,8 @@
         <origin xyz="0 0 -0.02" rpy="0 0 1.57" />
     </joint>
-    <joint name="depth_camera_base_joint" type="fixed">
-        <parent link="base_link"/>
-        <child link="depth_camera_link"/>
-        <origin xyz="0.155 0 0" rpy="-1.57 0 -1.57" />
+    <joint name="camera_camera_base_joint" type="fixed">
+        <parent link="base_link"/>
+        <child link="camera_camera_link"/>
+        <origin xyz="0.155 0 0.1" rpy="0 0 0" />
     </joint>
     <!-- Gazebo Plugins -->
@@ -349,4 +353,35 @@
     </sensor>
   </gazebo>
+  <gazebo reference="camera_camera_link">  <!-- replace with actual D435i base link -->
+    <sensor name="camera" type="depth">
+      <pose>0 0 0 0 0 0</pose>
+      <visualize>true</visualize>
+      <update_rate>5</update_rate>
+      <camera>
+        <horizontal_fov>1.39626</horizontal_fov> <!-- ~80 degrees -->
+        <image>
+          <width>640</width>
+          <height>480</height>
+          <format>R8G8B8</format>
+        </image>
+        <clip>
+          <near>0.1</near>
+          <far>10.0</far>
+        </clip>
+      </camera>
+      <plugin name="depth_camera" filename="libgazebo_ros_camera.so">
+        <!-- <camera_name>depth_camera</camera_name> -->
+        <frame_id>camera_camera_link</frame_id>
+        <!-- <image_topic>camera/depth/image_raw</image_topic>  Depth Image Topic -->
+        <!-- <depth_topic>camera/depth/image_raw</depth_topic>  Depth Image Topic -->
+        <!-- <point_cloud_topic>camera/depth/points</point_cloud_topic>  PointCloud2 Topic -->
+      </plugin>
+      <!-- Plugin to convert depth data into PointCloud2 -->
+      <!-- <plugin name="depth_camera_pointcloud" filename="libgazebo_ros_depth_camera.so">
+        <depth_image_topic>camera/depth/image_raw</depth_image_topic>
+        <point_cloud_topic>camera/depth/points</point_cloud_topic>
+      </plugin> -->
+    </sensor>
+  </gazebo>
   <!-- FRICTION AND PHYSICS -->
   <gazebo reference="wheel_FL_link">

Commit message: sim depth sensor still not fully working

File: src/simulation_package/urdf/leo_sim.urdf.xacro (robot description, xacro)
@@ -164,4 +164,5 @@
         </visual>
     </link>
+    <link name="camera_camera_frame_link" />
     <!-- JOINTS -->
     <joint name="base_footprint_joint" type="fixed">
@@ -208,4 +209,9 @@
         <child link="camera_camera_link"/>
         <origin xyz="0.155 0 0.1" rpy="0 0 0" />
+    </joint>
+    <joint name="camera_camera_frame_joint" type="fixed">
+        <parent link="camera_camera_link" />
+        <child link="camera_camera_frame_link" />
+        <origin xyz="0 0 0" rpy="-1.57 0 -1.57" />
     </joint>
     <!-- Gazebo Plugins -->
@@ -286,5 +292,5 @@
         </plugin>
   </gazebo>
-    <gazebo reference="base_link">
+  <gazebo reference="base_link">
     <sensor name="imu_sensor" type="imu">
       <topic>/model/leo_sim/imu</topic>
@@ -359,5 +365,5 @@
       <update_rate>5</update_rate>
       <camera>
-        <horizontal_fov>1.39626</horizontal_fov> <!-- ~80 degrees -->
+        <horizontal_fov>2</horizontal_fov> <!-- ~80 degrees -->
         <image>
           <width>640</width>
@@ -367,10 +373,11 @@
         <clip>
           <near>0.1</near>
-          <far>10.0</far>
+          <far>5.0</far>
         </clip>
       </camera>
       <plugin name="depth_camera" filename="libgazebo_ros_camera.so">
+        <!-- <ignition_frame_id>camera_camera_link</ignition_frame_id> -->
         <!-- <camera_name>depth_camera</camera_name> -->
-        <frame_id>camera_camera_link</frame_id>
+        <frame_name>camera_camera_frame_link</frame_name>
         <!-- <image_topic>camera/depth/image_raw</image_topic>  Depth Image Topic -->
         <!-- <depth_topic>camera/depth/image_raw</depth_topic>  Depth Image Topic -->

Commit message: point cloud data now works in rviz, not in nav yet

File: src/simulation_package/urdf/leo_sim.urdf.xacro (robot description, xacro)
@@ -157,5 +157,5 @@
     <link name="camera_camera_link">
         <visual>
-            <origin xyz="0 0 0" rpy="0.0 0.0 0.0"/>
+            <origin xyz="0 0 0" rpy="0 0 0"/>
             <geometry>
                 <box size="0.025 0.090 0.025"/>
@@ -208,10 +208,10 @@
         <parent link="base_link"/>
         <child link="camera_camera_link"/>
-        <origin xyz="0.155 0 0.1" rpy="0 0 0" />
+        <origin xyz="0.155 0 0.2" rpy="0 0 0" />
     </joint>
     <joint name="camera_camera_frame_joint" type="fixed">
         <parent link="camera_camera_link" />
         <child link="camera_camera_frame_link" />
-        <origin xyz="0 0 0" rpy="-1.57 0 -1.57" />
+        <origin xyz="0 0 0" rpy="1.57 3.14 1.57" />
     </joint>
     <!-- Gazebo Plugins -->
@@ -359,34 +359,26 @@
     </sensor>
   </gazebo>
-  <gazebo reference="camera_camera_link">  <!-- replace with actual D435i base link -->
-    <sensor name="camera" type="depth">
-      <pose>0 0 0 0 0 0</pose>
+  <gazebo reference="camera_camera_link">
+    <sensor name="depth_sensor" type="depth_camera">
+      <always_on>1</always_on>
       <visualize>true</visualize>
-      <update_rate>5</update_rate>
+      <update_rate>30</update_rate>
+      <frame_id>camera_camera_frame_link</frame_id>
+      <ignition_frame_id>camera_camera_frame_link</ignition_frame_id>
+      <topic>model/leo_sim/depth_camera</topic>
+      <optical_frame_id>camera_camera_frame_link</optical_frame_id>
       <camera>
-        <horizontal_fov>2</horizontal_fov> <!-- ~80 degrees -->
+        <horizontal_fov>1.51855</horizontal_fov>
+        <vertical_fov>1.01229</vertical_fov>
         <image>
-          <width>640</width>
-          <height>480</height>
+          <width>1280</width>
+          <height>720</height>
           <format>R8G8B8</format>
         </image>
         <clip>
-          <near>0.1</near>
-          <far>5.0</far>
+          <near>0.05</near>
+          <far>2.0</far>
         </clip>
       </camera>
-      <plugin name="depth_camera" filename="libgazebo_ros_camera.so">
-        <!-- <ignition_frame_id>camera_camera_link</ignition_frame_id> -->
-        <!-- <camera_name>depth_camera</camera_name> -->
-        <frame_name>camera_camera_frame_link</frame_name>
-        <!-- <image_topic>camera/depth/image_raw</image_topic>  Depth Image Topic -->
-        <!-- <depth_topic>camera/depth/image_raw</depth_topic>  Depth Image Topic -->
-        <!-- <point_cloud_topic>camera/depth/points</point_cloud_topic>  PointCloud2 Topic -->
-      </plugin>
-      <!-- Plugin to convert depth data into PointCloud2 -->
-      <!-- <plugin name="depth_camera_pointcloud" filename="libgazebo_ros_depth_camera.so">
-        <depth_image_topic>camera/depth/image_raw</depth_image_topic>
-        <point_cloud_topic>camera/depth/points</point_cloud_topic>
-      </plugin> -->
     </sensor>
   </gazebo>
